File: PCB_HW/STM32_DevBoard.kicad_sch (KiCad schematic)
At the start: 35 parts, among them J1 Conn_01x08_MountingPin, J2 Conn_01x04_MountingPin, J3 Conn_01x04_MountingPin, SW1 SW_Push, SW2 SW_Push, SW3 NRST, U1 STM32G031F6Px, U2 W25Q16JVSS, Y1 NX3215SA-32.768K

Commit message: Bus fix. "Connectors" sheet added
Parts:
- removed J1: Conn_01x08_MountingPin, Connector_Molex:Molex_PicoBlade_53261-0871_1x08-1MP_P1.25mm_Horizontal, symbol Connector_Generic_MountingPin:Conn_01x08_MountingPin
- removed J2: Conn_01x04_MountingPin, Connector_Molex:Molex_PicoBlade_53261-0471_1x04-1MP_P1.25mm_Horizontal, symbol Connector_Generic_MountingPin:Conn_01x04_MountingPin
- removed J3: Conn_01x04_MountingPin, Connector_PinHeader_2.54mm:PinHeader_1x04_P2.54mm_Vertical, symbol Connector_Generic_MountingPin:Conn_01x04_MountingPin
Connections:
- no-connect marks 3 -> 0
Other:
- added sheet Connectors (Connectors.kicad_sch)
- sheet USB ports: added {MainBus}; removed MainBus

Commit message: Some parts routed
Parts:
- added C15: 100nF, Capacitor_SMD:C_0603_1608Metric, symbol Device:C
- JP1, JP2, JP3, JP4, JP5, JP6, JP7, JP8, JP9: footprint Jumper:SolderJumper-2_P1.3mm_Open_TrianglePad1.0x1.5mm -> LocalLib:Jumper_0603
Connections:
- net +3.3V: now also C15.1
- net GNDD: now also C15.2
Other:
- moved on the sheet: R5, R8, SW1, SW2

Commit message: Fix
Parts:
- renumbered C15 to C3, C3 to C4, C4 to C5, C5 to C6
Changed lines of the file:
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@@
 		(dnp no)
 		(fields_autoplaced yes)
-		(property "Reference" "#PWR09"
+		(property "Reference" "#PWR010"
 			(at 149.86 106.68 0)
 			(effects
@@
 			(project "STM32_DevBoard"
 				(path "/b840a7da-4064-48df-a68c-9dffdf854821"
-					(reference "#PWR09")
+					(reference "#PWR010")
 					(unit 1)
 				)
@@
 		(dnp no)
 		(fields_autoplaced yes)
-		(property "Reference" "C15"
+		(property "Reference" "C3"
 			(at 274.32 88.8999 0)
 			(effects
@@
 			(project "STM32_DevBoard"
 				(path "/b840a7da-4064-48df-a68c-9dffdf854821"
-					(reference "C15")
+					(reference "C3")
 					(unit 1)
 				)
@@
 		(dnp no)
 		(fields_autoplaced yes)
-		(property "Reference" "#PWR012"
+		(property "Reference" "#PWR013"
 			(at 255.27 119.38 0)
 			(effects
@@
 			(project "STM32_DevBoard"
 				(path "/b840a7da-4064-48df-a68c-9dffdf854821"
-					(reference "#PWR012")
+					(reference "#PWR013")
 					(unit 1)
 				)
@@
 		(dnp no)
 		(fields_autoplaced yes)
-		(property "Reference" "#PWR010"
+		(property "Reference" "#PWR011"
 			(at 88.9 110.49 0)
 			(effects
@@
 			(project "STM32_DevBoard"
 				(path "/b840a7da-4064-48df-a68c-9dffdf854821"
-					(reference "#PWR010")
+					(reference "#PWR011")
 					(unit 1)
 				)
@@
 		(dnp no)
 		(fields_autoplaced yes)
-		(property "Reference" "#PWR011"
+		(property "Reference" "#PWR012"
 			(at 194.31 115.57 0)
 			(effects
@@
 			(project "STM32_DevBoard"
 				(path "/b840a7da-4064-48df-a68c-9dffdf854821"
-					(reference "#PWR011")
+					(reference "#PWR012")
 					(unit 1)
 				)
@@
 		(dnp no)
 		(fields_autoplaced yes)
-		(property "Reference" "#PWR08"
+		(property "Reference" "#PWR09"
 			(at 125.73 102.87 0)
 			(effects
@@
 			(project "STM32_DevBoard"
 				(path "/b840a7da-4064-48df-a68c-9dffdf854821"
-					(reference "#PWR08")
+					(reference "#PWR09")
 					(unit 1)
 				)
@@
 		(dnp no)
 		(fields_autoplaced yes)
-		(property "Reference" "#PWR056"
+		(property "Reference" "#PWR08"
 			(at 270.51 101.6 0)
 			(effects
@@
 			(project "STM32_DevBoard"
 				(path "/b840a7da-4064-48df-a68c-9dffdf854821"
-					(reference "#PWR056")
+					(reference "#PWR08")
 					(unit 1)
 				)
@@
 		(on_board yes)
 		(dnp no)
-		(property "Reference" "C3"
+		(property "Reference" "C4"
 			(at 81.28 95.25 0)
 			(effects
@@
 			(project "STM32_DevBoard"
 				(path "/b840a7da-4064-48df-a68c-9dffdf854821"
-					(reference "C3")
+					(reference "C4")
 					(unit 1)
 				)
@@
 		(on_board yes)
 		(dnp no)
-		(property "Reference" "C4"
+		(property "Reference" "C5"
 			(at 93.726 95.758 0)
 			(effects
@@
 			(project "STM32_DevBoard"
 				(path "/b840a7da-4064-48df-a68c-9dffdf854821"
-					(reference "C4")
+					(reference "C5")
 					(unit 1)
 				)
@@
 		(on_board yes)
 		(dnp no)
-		(property "Reference" "C5"
+		(property "Reference" "C6"
 			(at 196.596 99.06 0)
 			(effects
@@
 			(project "STM32_DevBoard"
 				(path "/b840a7da-4064-48df-a68c-9dffdf854821"
-					(reference "C5")
-					(unit 1)
-				)
+					(reference "C6")
+					(unit 1)
+				)
