File: PCB_HW/USB.kicad_sch (KiCad schematic)
At the start: 24 parts, among them J4 USB_C_Receptacle_USB2.0_16P, U3 SRV05-4, U4 ch343p, U5 AMS1117-3.3, U6 TLV62569DBV

Commit message: Bus fix. "Connectors" sheet added
Parts:
- added JP10: shunt, LocalLib:Jumper_0603, symbol Jumper:Jumper_2_Open
- added R14: 0.1, Resistor_SMD:R_0805_2012Metric, symbol Device:R
- added U6: MCP1700x-300xxTT, Package_TO_SOT_SMD:SOT-23, symbol Regulator_Linear:MCP1700x-300xxTT
- renumbered J4 to J1, R14 to R15, R15 to R16, U6 to U7
Connections:
- net +3.3V: now also JP10.2 (B), R14.2; no longer C11.1, C12.1, C8.1, L1.2, L2.2, R15.1, R9.2, U4.1 (VIO), U5.2 (VO)
- net +5V: now also U6.3 (VI)
- net GNDD: now also U6.1 (GND)
- new net +3.3V_sh: C11.1, C12.1, C8.1, JP10.1 (A), L1.2, L2.2, R14.1, R15.1, R9.2, U4.1 (VIO), U5.2 (VO), U6.2 (VO)
Other:
- moved on the sheet: C10, C11, C12, L2, R15, R16, U7

Commit message: Some parts routed
Parts:
- added C13: 100nF, Capacitor_SMD:C_0603_1608Metric, symbol Device:C
- added C14: 10uF, Capacitor_SMD:C_0805_2012Metric_Pad1.18x1.45mm_HandSolder, symbol Device:C
Connections:
- net +3.3V: now also C13.1, C14.1
- net GNDD: now also C13.2, C14.2

Commit message: Fix
Parts:
- renumbered C9 to C10, C14 to C11, C13 to C12, C10 to C13, C11 to C14, C12 to C15, C6 to C7, C7 to C8, C8 to C9
